File: Hardware/STM32withBle/STM32withBle.kicad_sch (KiCad schematic)
At the start: 40 parts, among them J1 USB_C_Receptacle_USB2.0_16P, J2 Conn_01x04_Pin, J3 Conn_ARM_SWD_TagConnect_TC2030, J4 Conn_Coaxial, SW1 SW_Push, U1 MIC5365-3.3YD5, U2 USBLC6-2SC6, U3 STM32WB55CEU6, X1 32kHz768, X2 32MHz

Commit message: Added the PDF File
Parts:
- added C19: 100n, Capacitor_SMD:C_0402_1005Metric, symbol Device:C
- C1, C15, C2, C5, C9: footprint (none) -> Capacitor_SMD:C_0603_1608Metric
- C10, C11, C12, C3, C4, C6, C7, C8: value 100nF -> 100n; footprint (none) -> Capacitor_SMD:C_0402_1005Metric
- C13, C14: value C -> 10p; footprint (none) -> Capacitor_SMD:C_0402_1005Metric
- C16: footprint (none) -> Capacitor_SMD:C_0402_1005Metric
- C17, C18: value C -> 0p8; footprint (none) -> Capacitor_SMD:C_0402_1005Metric
- D1: footprint (none) -> LED_SMD:LED_0402_1005Metric
- FLT1: footprint (none) -> STM32withBle_PCBFootprints:DLF162500LT-5028A1
- J1: footprint (none) -> Connector_USB:USB_C_Receptacle_GCT_USB4105-xx-A_16P_TopMnt_Horizontal
- J2: footprint (none) -> Connector_Molex:Molex_Mini-Fit_Sr_42820-42XX_1x04_P10.00mm_Horizontal
- J3: now in the parts list
- J4: footprint (none) -> Connector_Coaxial:U.FL_Hirose_U.FL-R-SMT-1_Vertical
- L1: value L -> 10n; footprint (none) -> Inductor_SMD:L_0402_1005Metric
- L2: value L -> 10u; footprint (none) -> Inductor_SMD:L_0805_2012Metric
- L3: value L -> 2n7; footprint (none) -> Inductor_SMD:L_0402_1005Metric
- R1, R2, R3, R4, R5, R6, R7: footprint (none) -> Resistor_SMD:R_0402_1005Metric
- SW1: footprint (none) -> Button_Switch_SMD:SW_SPST_CK_RS282G05A3
- X1: footprint (none) -> Crystal:Crystal_SMD_2012-2Pin_2.0x1.2mm
- X2: footprint (none) -> Crystal:Crystal_SMD_2016-4Pin_2.0x1.6mm
Connections:
- net GND: now also U2.2 (GND), C19.2
- net SWD_NRST: now also C19.1
